Commit message: error steady

File: sb_robot/manipulator.xacro (robot description, xacro)
@@ -150,4 +150,7 @@
             <origin xyz="${LINK1['position']}" rpy="${LINK1['orientation']}"/>
             <axis xyz="0 0 1"/>
+            <limit
+                velocity="0.5"
+                effort="0.5"/>
         </joint>
     </xacro:macro>
@@ -158,4 +161,7 @@
             <origin xyz="${LINK2['position']}" rpy="${LINK2['orientation']}"/>
             <axis xyz="0 0 1"/>
+            <limit
+                velocity="0.5"
+                effort="0.5"/>
         </joint>
     </xacro:macro>
