Commit message: add world

File: sb_robot/imusensor.xacro (robot description, xacro)
@@ -2,19 +2,19 @@
 <robot xmlns:xacro="http://www.ros.org/wiki/xacro">
     <xacro:macro name="imusensor" params="">
-        <gazebo reference="imusensor">
+        <gazebo reference="base_link">
             <gravity>true</gravity>
             <sensor name="imu_1" type="imu">
                 <always_on>true</always_on>
-                <update_rate>100</update_rate>
+                <update_rate>50</update_rate>
                 <visualize>true</visualize>
                 <topic>Imu_1</topic>
                 <plugin filename="libgazebo_ros_imu_sensor.so" name="imu_plugin">
                     <topicName>Imu_1</topicName>
-                    <bodyName>imusensor</bodyName>
-                    <updateRateHZ>10.0</updateRateHZ>
+                    <bodyName>base_link</bodyName>
+                    <updateRateHZ>50.0</updateRateHZ>
                     <gaussianNoise>0.0</gaussianNoise>
                     <xyzOffset>0 0 0</xyzOffset>
                     <rpyOffset>0 0 0</rpyOffset>
-                    <frameName>imusensor</frameName>
+                    <frameName>base_link</frameName>
                     <initialOrientationAsReference>false</initialOrientationAsReference>
                 </plugin>

File: sb_robot/manipulator.xacro (robot description, xacro)
@@ -33,8 +33,8 @@
             <surface>
             <friction>
-            <ode>
-                <mu>100</mu>
-                <mu2>100</mu2>
-            </ode>
+                <ode>
+                    <mu>1000</mu>
+                    <mu2>1000</mu2>
+                </ode>
             </friction>
         </surface>
@@ -150,7 +150,4 @@
             <origin xyz="${LINK1['position']}" rpy="${LINK1['orientation']}"/>
             <axis xyz="0 0 1"/>
-            <limit
-                velocity="0.5"
-                effort="0.5"/>
         </joint>
     </xacro:macro>
@@ -161,7 +158,4 @@
             <origin xyz="${LINK2['position']}" rpy="${LINK2['orientation']}"/>
             <axis xyz="0 0 1"/>
-            <limit
-                velocity="0.5"
-                effort="0.5"/>
         </joint>
     </xacro:macro>
@@ -174,5 +168,5 @@
     </xacro:macro>
     <xacro:macro name="self_balancing" params="">
-        <link name="base"/>
+        <!-- <link name="base"/> -->
         <link name="base_link">
             <xacro:base_visual />
@@ -190,13 +184,13 @@
             <xacro:link2_collision />
         </link>
-        <link name="imusensor">
+        <!-- <link name="imusensor">
             <xacro:imusensor_visual/>
             <xacro:imusensor_inertial />
             <xacro:imusensor_collision/>
-        </link>
-        <xacro:base />
+        </link> -->
+        <!-- <xacro:base /> -->
         <xacro:joint0 />
         <xacro:joint1 />
-        <xacro:sensor_joint />
+        <!-- <xacro:sensor_joint /> -->
     </xacro:macro>
 </robot>
